File: CarbonAwareCircuit.kicad_sch (KiCad schematic)
At the start: 12 parts, among them J1 USB_C_Receptacle_USB2.0_14P, SW1 SW_Push, U1 LD1117V, U2 ESP32-C3-WROOM-02

Commit message: eeschema done
Parts:
- added J2: USB_A, symbol Connector:USB_A
- added Q1: AO3401A, Package_TO_SOT_SMD:SOT-23, symbol Transistor_FET:AO3401A
- added SW2: SW_Push, symbol Switch:SW_Push
Connections:
- net at C1.2, D1.1 (K), J1.A1 (GND)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: now also J2.4 (GND), J2.SH (Shield)
- net at R6.1, U2.2 (EN): now also SW2.1; no longer C1.1
- net at U2.3 (IO4): now also Q1.1 (G)
- net at J1.A4 (VBUS), J1.A9 (VBUS), J1.B4 (VBUS)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: now also Q1.2 (S)
- new net: C1.1, SW2.2
- new net: J2.1 (VBUS), Q1.3 (D)
- new net: J2.2 (D-), J2.3 (D+)
Other:
- moved on the sheet: C1, D1, J1, R1, R2, R3, R5, R6, SW1, U1, U2

Commit message: massive strides in pcbnew
Parts:
- removed C1: 1µF, symbol Device:C_Small
- D1: footprint (none) -> LED_THT:LED_D3.0mm_Horizontal_O1.27mm_Z2.0mm_Clear
- J2: footprint (none) -> Connector_USB:USB_A_CNCTech_1001-011-01101_Horizontal
- R1, R2, R3, R4, R5, R6: footprint (none) -> Resistor_THT:R_Axial_DIN0207_L6.3mm_D2.5mm_P15.24mm_Horizontal
- SW1: footprint (none) -> Button_Switch_THT:SW_PUSH_6mm_H4.3mm
- SW2: footprint (none) -> Button_Switch_THT:SW_PUSH_6mm_H7.3mm
Connections:
- net at D1.1 (K), J1.A1 (GND), J1.A12 (GND)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: now also SW2.2
Other:
- company: (none) -> Abhiram Vadali
Changed lines of the file:
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@@
 		(date "2026-04-08")
 		(rev "1.0")
+		(company "Abhiram Vadali")
+		(comment 1 "Used in STEAM ICAC 2026 - Team C6")
 	)
 	(junction
@@
 	(wire
 		(pts
-			(xy 208.28 138.43) (xy 208.28 105.41)
+			(xy 208.28 105.41) (xy 208.28 147.32)
 		)
 		(stroke
@@
 		(pts
 			(xy 210.82 139.7) (xy 210.82 154.94)
-		)
-		(stroke
-			(width 0)
-			(type default)
-		)
-	)
-	(wire
-		(pts
-			(xy 208.28 147.32) (xy 208.28 143.51)
 		)
 		(stroke
@@
 			)
 		)
-		(property "Footprint" ""
+		(property "Footprint" "Resistor_THT:R_Axial_DIN0207_L6.3mm_D2.5mm_P15.24mm_Horizontal"
 			(at 222.25 127 0)
 			(hide yes)
@@
 			)
 		)
-		(property "Footprint" ""
+		(property "Footprint" "Button_Switch_THT:SW_PUSH_6mm_H7.3mm"
 			(at 214.63 152.4 0)
 			(hide yes)
@@
 			)
 		)
-		(property "Footprint" ""
+		(property "Footprint" "Resistor_THT:R_Axial_DIN0207_L6.3mm_D2.5mm_P15.24mm_Horizontal"
 			(at 205.74 100.33 0)
 			(hide yes)
@@
 			)
 		)
-		(property "Footprint" ""
+		(property "Footprint" "Resistor_THT:R_Axial_DIN0207_L6.3mm_D2.5mm_P15.24mm_Horizontal"
 			(at 219.71 139.7 0)
 			(hide yes)
@@
 			)
 		)
-		(property "Footprint" ""
+		(property "Footprint" "Button_Switch_THT:SW_PUSH_6mm_H4.3mm"
 			(at 214.63 116.84 0)
 			(hide yes)
@@
 			)
 		)
-		(property "Footprint" ""
+		(property "Footprint" "Resistor_THT:R_Axial_DIN0207_L6.3mm_D2.5mm_P15.24mm_Horizontal"
 			(at 215.9 124.46 0)
 			(hide yes)
@@
 			)
 		)
-		(property "Footprint" ""
+		(property "Footprint" "Resistor_THT:R_Axial_DIN0207_L6.3mm_D2.5mm_P15.24mm_Horizontal"
 			(at 201.93 105.41 0)
 			(hide yes)
@@
 				(path "/997ad0de-87ea-4de7-b67f-c27fa67242e9"
 					(reference "R1")
-					(unit 1)
-				)
-			)
-		)
-	)
-	(symbol
-		(lib_id "Device:C_Small")
-		(at 208.28 140.97 180)
-		(unit 1)
-		(body_style 1)
-		(exclude_from_sim no)
-		(in_bom yes)
-		(on_board yes)
-		(in_pos_files yes)
-		(dnp no)
-		(fields_autoplaced yes)
-		(property "Reference" "C1"
-			(at 201.93 140.9637 90)
-			(show_name no)
-			(do_not_autoplace no)
-			(effects
-				(font
-					(size 1.27 1.27)
-				)
-			)
-		)
-		(property "Value" "1µF"
-			(at 204.47 140.9637 90)
-			(show_name no)
-			(do_not_autoplace no)
-			(effects
-				(font
-					(size 1.27 1.27)
-				)
-			)
-		)
-		(property "Footprint" ""
-			(at 208.28 140.97 0)
-			(hide yes)
-			(show_name no)
-			(do_not_autoplace no)
-			(effects
-				(font
-					(size 1.27 1.27)
-				)
-			)
-		)
-		(property "Datasheet" ""
-			(at 208.28 140.97 0)
-			(hide yes)
-			(show_name no)
-			(do_not_autoplace no)
-			(effects
-				(font
-					(size 1.27 1.27)
-				)
-			)
-		)
-		(property "Description" "Unpolarized capacitor, small symbol"
-			(at 208.28 140.97 0)
-			(hide yes)
-			(show_name no)
-			(do_not_autoplace no)
-			(effects
-				(font
-					(size 1.27 1.27)
-				)
-			)
-		)
-		(pin "2"
-		)
-		(pin "1"
-		)
-		(instances
-			(project "CarbonAwareCircuit"
-				(path "/997ad0de-87ea-4de7-b67f-c27fa67242e9"
-					(reference "C1")
 					(unit 1)
 				)
@@
 			)
 		)
-		(property "Footprint" ""
+		(property "Footprint" "LED_THT:LED_D3.0mm_Horizontal_O1.27mm_Z2.0mm_Clear"
 			(at 217.17 127 0)
 			(hide yes)
@@
 			)
 		)
-		(property "Footprint" ""
+		(property "Footprint" "Connector_USB:USB_A_CNCTech_1001-011-01101_Horizontal"
 			(at 158.75 144.78 0)
 			(hide yes)
@@
 			)
 		)
-		(property "Footprint" ""
+		(property "Footprint" "Resistor_THT:R_Axial_DIN0207_L6.3mm_D2.5mm_P15.24mm_Horizontal"
 			(at 218.44 149.86 0)
 			(hide yes)
