File: CarbonAwareCircuit.kicad_sch (KiCad schematic)
At the start: 14 parts, among them J1 USB_C_Receptacle_USB2.0_14P, J2 USB_A, Q1 AO3401A, SW1 SW_Push, SW2 SW_Push, U1 LD1117V, U2 ESP32-C3-WROOM-02

Commit message: changed output to female
Parts:
- J2: footprint Connector_USB:USB_A_CNCTech_1001-011-01101_Horizontal -> Connector_USB:USB_A_Receptacle_GCT_USB1046
Changed lines of the file:
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@@
 			)
 		)
-		(property "Footprint" "Connector_USB:USB_A_CNCTech_1001-011-01101_Horizontal"
+		(property "Footprint" "Connector_USB:USB_A_Receptacle_GCT_USB1046"
 			(at 158.75 144.78 0)
 			(hide yes)
