File: CarbonAwareCircuit.kicad_pcb (KiCad board)
At the start: 2 copper layers, 64 x 55.5 mm, 15 parts, among them J1 USB_C_Receptacle_USB2.0_14P, J2 USB_A, Q1 AO3401A, SW1 SW_Push, SW2 SW_Push, U1 LD1117V, U2 ESP32-C3-WROOM-02

Commit message: changed output to female
Parts:
- J2: footprint Connector_USB:USB_A_CNCTech_1001-011-01101_Horizontal -> Connector_USB:USB_A_Receptacle_GCT_USB1046
- turned J2 to 180 degrees
Routing:
- net Net-(D1-K): track 143.6 -> 151.8 mm, vias 2 -> 3
- net Net-(J2-VBUS): track 9.13 -> 16.9 mm
Other:
- board size 64 x 55.5 mm -> 64 x 52.5 mm
